File: NixieIndicator.kicad_pcb (KiCad board)
At the start: 2 copper layers, 168 x 50 mm, 70 parts, among them J1 Conn_01x03_Pin, J2 RIGHT, J3 MIDDLE, J4 LEFT, J5 Conn_01x12_Pin, J6 I2C, J7 EUSART, J8 Conn_01x04_Pin, Q1 MPSA42, Q2 MPSA42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

Commit message: 製造後データを追加
Parts:
- added R37: 100k, Resistor_THT:R_Axial_DIN0207_L6.3mm_D2.5mm_P10.16mm_Horizontal, F.Cu at (12.1, 15.9)
- added R39: 100k, Resistor_THT:R_Axial_DIN0207_L6.3mm_D2.5mm_P10.16mm_Horizontal, F.Cu at (44.5, 15.9)
- added R41: 100k, Resistor_THT:R_Axial_DIN0207_L6.3mm_D2.5mm_P10.16mm_Horizontal, F.Cu at (78.9, 9.10)
- moved U5 2.56 mm to (23.3, 24.6)
- moved R38 2.40 mm to (15.1, 15.9)
- moved C1 2.40 mm to (20.6, 22.5)
- moved C3 2.40 mm to (20.6, 25.0)
- moved Q1 2.40 mm to (19.6, 19.3)
- renumbered R37 to R38, R38 to R40, R39 to R42
Connections:
- Q1 pad 2: /DOT_2 -> Net-(Q1-B)
- Q2 pad 2: /DOT_1 -> Net-(Q2-B)
- Q3 pad 2: /DOT_0 -> Net-(Q3-B)
Routing:
- net Net-(Q3-B): track 0.00 -> 14.8 mm
- net /DOT_0: track 44.5 -> 56.2 mm, vias 3 -> 2
- net Net-(Q1-B): track 0.00 -> 8.36 mm
- net Net-(Q2-B): track 0.00 -> 8.36 mm
- net /DEC2_1: track 12.7 -> 17.9 mm
- net /5V: track 273.7 -> 278.8 mm, vias 9 -> 7
- net /DEC2_6: track 26.5 -> 21.6 mm
- net /DEC2_9: track 25.5 -> 21.5 mm
- net /DEC2_C: track 31.7 -> 28.3 mm
- net /DEC2_B: track 25.6 -> 22.4 mm, vias 2 -> 0
- net /DEC2_8: track 19.8 -> 16.6 mm, vias 2 -> 0
- net /DEC2_D: track 27.3 -> 24.5 mm, vias 2 -> 0
- net /DEC2_A: track 25.4 -> 27.8 mm
- net /DEC2_3: track 20.8 -> 18.7 mm
- net GND: track 294.3 -> 296.3 mm, vias 235 -> 290
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Other:
- board text added: "JLCJLCJLCJLC"
- board text added: "RC5 RD1 RD2 RD3"
