File: NixieIndicator.kicad_sch (KiCad schematic)
At the start: 62 parts, among them J1 Conn_01x03_Pin, J2 Conn_01x12_Pin, J3 Conn_01x12_Pin, J4 Conn_01x12_Pin, J5 Conn_01x12_Pin, J6 Conn_01x03_Pin, J7 Conn_01x03_Pin, J8 Conn_01x04_Pin, Q1 MPSA42, Q2 MPSA42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

Commit message: 製造後データを追加
Parts:
- added R37, R39, R41: 100k, Resistor_THT:R_Axial_DIN0207_L6.3mm_D2.5mm_P10.16mm_Horizontal, symbol Device:R
- J2: value Conn_01x12_Pin -> RIGHT
- J3: value Conn_01x12_Pin -> MIDDLE
- J4: value Conn_01x12_Pin -> LEFT
- J6: value Conn_01x03_Pin -> I2C
- J7: value Conn_01x03_Pin -> EUSART
- U2, U3, U4: value TLP627-4 -> TLP627
- renumbered R37 to R38, R38 to R40, R39 to R42
Connections:
- net DOT_0: now also R41.2; no longer Q3.2 (B)
- net DOT_1: now also R39.2; no longer Q2.2 (B)
- net DOT_2: now also R37.2; no longer Q1.2 (B)
- new net: Q2.2 (B), R39.1
- new net: Q3.2 (B), R41.1
- new net: Q1.2 (B), R37.1
